Commit message: 2025.5.10

File: src/1410_URDF_test2/urdf/1410_URDF_test2.urdf (robot description, URDF)
Before this commit: robot 1410_URDF_test2, 8 links, 7 joints
Links:
- link base_link: mass 0.001 -> 0.1
- link link_1: mass 0.001 -> 0.1
- link link_2: mass 0.001 -> 0.1
- link link_3: mass 0.001 -> 0.1
- link link_4: mass 0.001 -> 0.1
- link link_5: mass 0.001 -> 0.1
- link link_6: mass 0.001 -> 0.1
