Commit message: update readme and gazebo

File: src/1410_URDF_test2/urdf/1410_URDF_ik.urdf (robot description, URDF)
Before this commit: robot 1410_URDF_test2, 7 links, 6 joints
Links:
- added link world
Joints:
- added joint world_to_base_link: type fixed, parent world, child base_link

File: src/1410_URDF_test2/urdf/1410_URDF_test2.urdf (robot description, URDF)
Before this commit: robot 1410_URDF_test2, 8 links, 7 joints
Links:
- link base_link: mass 0.1 -> 25.458
- link link_1: mass 0.1 -> 31.968
- link link_2: mass 0.1 -> 7.6192
- link link_3: mass 0.1 -> 7.4587
- link link_4: mass 0.1 -> 11.023
- link link_5: mass 0.1 -> 0.29435
- link link_6: mass 0.1 -> 0.016853
Joints:
- joint joint_1: limit lower=-5.933 upper=5.933 effort=50 velocity=50 -> lower=-2.96 upper=2.96 effort=50 velocity=50
- joint joint_2: limit lower=-2.443 upper=2.443 effort=50 velocity=50 -> lower=-1.22 upper=1.22 effort=50 velocity=50
- joint joint_3: limit lower=-2.3557 upper=2.3557 effort=50 velocity=50 -> lower=-1.22 upper=1.22 effort=50 velocity=50
- joint joint_4: limit lower=-5.235 upper=5.235 effort=50 velocity=50 -> lower=-2.617 upper=2.617 effort=50 velocity=50
- joint joint_5: limit lower=-4.0135 upper=4.0135 effort=50 velocity=50 -> lower=-2 upper=2 effort=50 velocity=50
- joint joint_6: limit lower=-6.282 upper=6.282 effort=50 velocity=50 -> lower=-5.235 upper=5.235 effort=50 velocity=50
